File: MESC_18_FET_THROUGH/MESC_18_FET_THROUGH/MESC_18_FET_THROUGH.kicad_pcb (KiCad board)
At the start: 4 copper layers, 100 x 50 mm, 118 parts, among them J1 Conn_01x01_Male, J2 Conn_01x01_Male, J3 Conn_01x01_Male, J4 Conn_01x01_Male, J5 Conn_01x01_Male, J6 Conn_01x01_Male, J7 Conn_01x08_Male, J8 Conn_01x08_Male, J9 Conn_01x08_Male, Q1 IRLZ44N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

Commit message: Add DC bus voltage output to power board.
Parts:
- C1, C11, C12, C13, C14, C15, C16, C2, C21, C22, C23, C24, C25, C26, C3, C4, C5, C6: value C_Small -> DNF 4.7nF 25V
- C10, C17, C18, C19, C20, C27, C28, C29, C30, C37, C7, C8, C9: value C_Small -> 1uF 100V
- C36, C38, C39: value C_Small -> 4.7nF 100V
- J1, J2, J3, J4, J5, J6: value Conn_01x01_Male -> M4 screw
- Q1, Q10, Q11, Q12, Q13, Q14, Q15, Q16, Q17, Q18, Q2, Q3, Q4, Q5, Q6, Q7, Q8, Q9: value IRLZ44N -> STP150N10F7
- R1, R10, R11, R13, R14, R16, R17, R19, R20, R22, R23, R25, R26, R3, R4, R5, R7, R8: value R_Small -> 4.7R
- R12, R15, R18, R2, R21, R24, R27, R28, R31, R32, R33, R34, R35, R36, R37, R38, R6, R9: value R_Small -> 0R001
- R29, R30, R39, R40, R41, R42: value R_Small -> DNF 100R
- R43, R44, R45: value R_Small -> 2R2
Connections:
- J7 pad 8: Net-(J7-Pad8) -> +VDC
Routing:
- net +VDC: track 0.00 -> 46.2 mm, vias 0 -> 1
